File: hardware/malenki-hv/motor_driver.kicad_sch (KiCad schematic)
At the start: 3 parts, among them J4 Conn_01x02_Male-Connector, U4 DRV8231DSGR

Commit message: Updated u1 QFN symbol by adding solder paste layer, minor schematic updates to fix check errors, converted to kiCad 9, Updated BOM with LSCS numbers, fixed BOM errors.
Parts:
- C1: MPN (none) -> CL10A106MA8NRNC
- U4: MPN (none) -> DRV8231DSGR; Manufacturer (none) -> TI
